File: camara-diy.kicad_pcb (KiCad board)
At the start: 2 copper layers, 17 parts, among them J1 Conn_01x07, J3 Conn_01x02, SW1 SW_Push, SW2 SW_Push, U1 XIAO-ESP32-S3-SMD, U2 TP4056-42-ESOP8

Commit message: archivos + pcb actualizados
Parts:
- added 10uF1: C6, Capacitor_SMD:C_0805_2012Metric, F.Cu at (174.5, 119.5)
- added R3: 2k, Resistor_SMD:R_0402_1005Metric, F.Cu at (179.5, 118.5)
- 100nF1: value C -> C5
- 10uF2: value C -> C7
- moved J3 25.2 mm to (205.5, 117.5)
- moved R1 23.8 mm to (174.5, 126.5)
- moved R2 23.0 mm to (170.3, 126.5)
- moved 10uF2 13.7 mm to (206.5, 126.2)
- moved J1 1.50 mm to (206.5, 93.5)
- moved D3 0.80 mm to (196.0, 118.2)
- moved D2 0.28 mm to (188.0, 126.2)
- moved D1 0.19 mm to (182.5, 126.2)
- renumbered R11k1 to R1, R21k1 to R2
Connections:
- 100nF1 pad 2: +3V3 -> GND
- 10uF2 pad 2: +3V3 -> GND
- C1 pad 2: +3V3 -> GND
- C2 pad 2: +3V3 -> GND
- C3 pad 2: +3V3 -> GND
- C4 pad 2: +3V3 -> GND
- D1 pad 1: +3V3 -> GND
- D2 pad 1: +3V3 -> GND
- D2 pad 2: +3V3 -> Net-(D2-A)
- J1 pad 2: +3V3 -> GND
- J3 pad 2: +3V3 -> GND
- R2 pad 1: +3V3 -> Net-(D2-A)
- R2 pad 2: +3V3 -> Net-(U2-~{STDBY})
- SW1 pad 2: +3V3 -> GND
- SW2 pad 2: +3V3 -> GND
- U1 pad 13: +3V3 -> GND
- U2 pad 1: +3V3 -> GND
- U2 pad 2: +3V3 -> Net-(U2-PROG)
- U2 pad 3: +3V3 -> GND
- U2 pad 6: +3V3 -> Net-(U2-~{STDBY})
- U2 pad 9: +3V3 -> GND
Routing:
- net +5V: track 0.00 -> 151.6 mm
- net +3V3: track 0.00 -> 117.5 mm
- net /BAT_18650: track 0.00 -> 81.5 mm
- net /SPI_MOSI: track 0.00 -> 63.8 mm
- net Net-(U2-~{STDBY}): track 0.00 -> 54.6 mm
- net Net-(U2-~{CHRG}): track 0.00 -> 53.6 mm
- net /BTN_MODO: track 0.00 -> 35.5 mm
- net /DISP_CS: track 0.00 -> 32.6 mm
- net /DISP_DC: track 0.00 -> 28.4 mm
- net /BTN_SHUTTER: track 0.00 -> 23.0 mm
- net Net-(D2-A): track 0.00 -> 20.3 mm
- net /SPI_CLK: track 0.00 -> 13.1 mm
- net /DISP_RES: track 0.00 -> 10.8 mm
- net Net-(D1-A): track 0.00 -> 10.1 mm
- net Net-(U2-PROG): track 0.00 -> 2.85 mm
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- added copper zone on B.Cu, net GND
Other:
- board outline added: 59.5 x 47 mm
